Commit message: visualized nano hand in rviz; still need to prevent collision

File: ros_ws/src/hands/urdf/nano/nano_hand_right_backup.urdf (robot description, URDF)
Before this commit: robot nanohand, 22 links, 21 joints
Links:
- removed link base
Joints:
- removed joint palm_to_base

Commit message: nano IK almost works; need to fix jerky thumb, self collision, limit too strict

File: ros_ws/src/hands/urdf/nano/nano_hand_right_backup.urdf (robot description, URDF)
Before this commit: robot nanohand, 21 links, 20 joints
Links:
- added link base
Joints:
- added joint palm_to_base: type fixed, parent palm, child base, origin xyz=0 0 0 rpy=3.141592653589793 0 0

File: ros_ws/src/hands/urdf/nano/nano_hand_right_original.urdf (robot description, URDF)
Before this commit: robot nanohand, 22 links, 21 joints
Links:
- removed link base
Joints:
- removed joint palm_to_base
- joint index_curl: limit lower=0.0 upper=1.06 effort=1.0 velocity=3.0 -> lower=0.0 upper=1.57 effort=1.0 velocity=3.0
- joint index_curl_dip: limit lower=0.0 upper=1.64 effort=1.0 velocity=3.0 -> lower=0.0 upper=1.57 effort=1.0 velocity=3.0; mimic joint=index_curl multiplier=2.23 offset=0.0 -> joint=index_curl multiplier=0.5 offset=0.0
- joint index_curl_pip: limit lower=0.0 upper=1.65 effort=1.0 velocity=3.0 -> lower=0.0 upper=1.57 effort=1.0 velocity=3.0; mimic joint=index_curl multiplier=2 offset=0.0 -> joint=index_curl multiplier=0.7 offset=0.0
- joint index_wiggle: limit lower=-0.17 upper=0.17 effort=1.0 velocity=3.0 -> lower=-0.256 upper=0.256 effort=1.0 velocity=3.0
- joint middle_curl: limit lower=0.0 upper=1.09 effort=1.0 velocity=3.0 -> lower=0.0 upper=1.57 effort=1.0 velocity=3.0
- joint middle_curl_dip: limit lower=0.0 upper=1.6 effort=1.0 velocity=3.0 -> lower=0.0 upper=1.57 effort=1.0 velocity=3.0; mimic joint=middle_curl multiplier=2.18 offset=0.0 -> joint=middle_curl multiplier=2.85 offset=0.0
- joint middle_curl_pip: limit lower=0.0 upper=1.65 effort=1.0 velocity=3.0 -> lower=0.0 upper=1.57 effort=1.0 velocity=3.0; mimic joint=middle_curl multiplier=2 offset=0.0 -> joint=middle_curl multiplier=2.2 offset=0.0
- joint middle_wiggle: limit lower=-0.13 upper=0.24 effort=1.0 velocity=3.0 -> lower=-0.256 upper=0.256 effort=1.0 velocity=3.0
- joint pinky_curl: limit lower=0.0 upper=0.97 effort=1.0 velocity=3.0 -> lower=0.0 upper=1.57 effort=1.0 velocity=3.0
- joint pinky_curl_dip: limit lower=0.0 upper=1.64 effort=1.0 velocity=3.0 -> lower=0.0 upper=1.57 effort=1.0 velocity=3.0; mimic joint=pinky_curl multiplier=2.23 offset=0.0 -> joint=pinky_curl multiplier=3.94 offset=0.0
- joint pinky_curl_pip: limit lower=0.0 upper=1.41 effort=1.0 velocity=3.0 -> lower=0.0 upper=1.57 effort=1.0 velocity=3.0; mimic joint=pinky_curl multiplier=2 offset=0.0 -> joint=pinky_curl multiplier=2.92 offset=0.0
- joint pinky_wiggle: limit lower=-0.17 upper=0.26 effort=1.0 velocity=3.0 -> lower=-0.256 upper=0.256 effort=1.0 velocity=3.0
- joint ring_curl: limit lower=0.0 upper=0.83 effort=1.0 velocity=3.0 -> lower=0.0 upper=1.57 effort=1.0 velocity=3.0
- joint ring_curl_dip: limit lower=0.0 upper=1.55 effort=1.0 velocity=3.0 -> lower=0.0 upper=1.57 effort=1.0 velocity=3.0; mimic joint=ring_curl multiplier=1.96 offset=0.0 -> joint=ring_curl multiplier=2.85 offset=0.0
- joint ring_curl_pip: limit lower=0.0 upper=1.29 effort=1.0 velocity=3.0 -> lower=0.0 upper=1.57 effort=1.0 velocity=3.0; mimic joint=ring_curl multiplier=1.5 offset=0.0 -> joint=ring_curl multiplier=2.31 offset=0.0
- joint ring_wiggle: limit lower=-0.2 upper=0.07 effort=1.0 velocity=3.0 -> lower=-0.256 upper=0.256 effort=1.0 velocity=3.0
- joint thumb_curl: limit lower=0.0 upper=0.68 effort=1.0 velocity=3.0 -> lower=0.0 upper=1.57 effort=1.0 velocity=3.0
- joint thumb_curl_dip: limit lower=0.0 upper=1.65 effort=1.0 velocity=3.0 -> lower=0.0 upper=1.57 effort=1.0 velocity=3.0; mimic joint=thumb_curl multiplier=2 offset=0.0 -> joint=thumb_curl multiplier=0.54 offset=0.0
- joint thumb_curl_pip: limit lower=0.0 upper=0.66 effort=1.0 velocity=3.0 -> lower=0.0 upper=1.57 effort=1.0 velocity=3.0; mimic joint=thumb_curl multiplier=0.83 offset=0.0 -> joint=thumb_curl multiplier=0.71 offset=0.0
- joint thumb_wiggle: limit lower=-0.78 upper=1.48 effort=1.0 velocity=3.0 -> lower=-1.3 upper=1.3 effort=1.0 velocity=3.0
