Commit message: added meshes & fixed paths

File: ros_ws/src/hands/urdf/nano/nano_hand_right.urdf (robot description, URDF)
Before this commit: robot nanohand, 21 links, 20 joints
Links:
- link index_knuckle: geometry collision mesh filename=package://hands/urdf/nano/meshes/Index_knuckle_section.stl; visual mesh filename=package://hands/urdf/nano/meshes/Index_knuckle_section.stl
- link index_mid: geometry collision mesh filename=package://hands/urdf/nano/meshes/Index_mid_section.stl; visual mesh filename=package://hands/urdf/nano/meshes/Index_mid_section.stl
- link index_tip: geometry collision mesh filename=package://hands/urdf/nano/meshes/Index_tip_section.stl; visual mesh filename=package://hands/urdf/nano/meshes/Index_tip_section.stl
- link middle_knuckle: geometry collision mesh filename=package://hands/urdf/nano/meshes/Middle_knuckle_section.stl; visual mesh filename=package://hands/urdf/nano/meshes/Middle_knuckle_section.stl
- link middle_mid: geometry collision mesh filename=package://hands/urdf/nano/meshes/Middle_mid_section.stl; visual mesh filename=package://hands/urdf/nano/meshes/Middle_mid_section.stl
- link middle_tip: geometry collision mesh filename=package://hands/urdf/nano/meshes/Middle_tip_section.stl; visual mesh filename=package://hands/urdf/nano/meshes/Middle_tip_section.stl
- link palm: geometry collision mesh filename=package://hands/urdf/nano/meshes/palm.stl; visual mesh filename=package://hands/urdf/nano/meshes/palm.stl
- link pinky_knuckle: geometry collision mesh filename=package://hands/urdf/nano/meshes/Pinky_knuckle_section.stl; visual mesh filename=package://hands/urdf/nano/meshes/Pinky_knuckle_section.stl
- link pinky_mid: geometry collision mesh filename=package://hands/urdf/nano/meshes/Pinky_mid_section.stl; visual mesh filename=package://hands/urdf/nano/meshes/Pinky_mid_section.stl
- link pinky_tip: geometry collision mesh filename=package://hands/urdf/nano/meshes/Pinky_tip_section.stl; visual mesh filename=package://hands/urdf/nano/meshes/Pinky_tip_section.stl
- link ring_knuckle: geometry collision mesh filename=package://hands/urdf/nano/meshes/Ring_knuckle_section.stl; visual mesh filename=package://hands/urdf/nano/meshes/Ring_knuckle_section.stl
- link ring_mid: geometry collision mesh filename=package://hands/urdf/nano/meshes/Ring_mid_section.stl; visual mesh filename=package://hands/urdf/nano/meshes/Ring_mid_section.stl
- link ring_tip: geometry collision mesh filename=package://hands/urdf/nano/meshes/Ring_tip_section.stl; visual mesh filename=package://hands/urdf/nano/meshes/Ring_tip_section.stl
- link thumb_knuckle: geometry collision mesh filename=package://hands/urdf/nano/meshes/Thumb_knuckle_section.stl; visual mesh filename=package://hands/urdf/nano/meshes/Thumb_knuckle_section.stl
- link thumb_mid: geometry collision mesh filename=package://hands/urdf/nano/meshes/Thumb_mid_section.stl; visual mesh filename=package://hands/urdf/nano/meshes/Thumb_mid_section.stl
- link thumb_tip: geometry collision mesh filename=package://hands/urdf/nano/meshes/Thumb_tip_section.stl; visual mesh filename=package://hands/urdf/nano/meshes/Thumb_tip_section.stl
Joints:
- joint middle_curl_dip: mimic joint=middle_curl multiplier=0.5 offset=0.0 -> joint=middle_curl multiplier=2.85 offset=0.0
- joint middle_curl_pip: mimic joint=middle_curl multiplier=0.7 offset=0.0 -> joint=middle_curl multiplier=2.2 offset=0.0
- joint pinky_curl_dip: mimic joint=pinky_curl multiplier=0.5 offset=0.0 -> joint=pinky_curl multiplier=3.94 offset=0.0
- joint pinky_curl_pip: mimic joint=pinky_curl multiplier=0.7 offset=0.0 -> joint=pinky_curl multiplier=2.92 offset=0.0
- joint ring_curl_dip: mimic joint=ring_curl multiplier=0.5 offset=0.0 -> joint=ring_curl multiplier=2.85 offset=0.0
- joint ring_curl_pip: mimic joint=ring_curl multiplier=0.7 offset=0.0 -> joint=ring_curl multiplier=2.31 offset=0.0
- joint thumb_curl_dip: mimic joint=thumb_curl multiplier=0.5 offset=0.0 -> joint=thumb_curl multiplier=0.54 offset=0.0
- joint thumb_curl_pip: mimic joint=thumb_curl multiplier=0.7 offset=0.0 -> joint=thumb_curl multiplier=0.71 offset=0.0
- joint thumb_wiggle: limit lower=-0.5 upper=0.5 effort=1.0 velocity=3.0 -> lower=-1.3 upper=1.3 effort=1.0 velocity=3.0

Commit message: IK for all fingers; lower thumb DIP multiplier

File: ros_ws/src/hands/urdf/nano/nano_hand_right.urdf (robot description, URDF)
Before this commit: robot nanohand, 22 links, 21 joints
Joints:
- joint thumb_curl_dip: mimic joint=thumb_curl multiplier=2 offset=0.0 -> joint=thumb_curl multiplier=1 offset=0.0

Commit message: added fingertip joints; fingers moved slightly less

File: ros_ws/src/hands/urdf/nano/nano_hand_right.urdf (robot description, URDF)
Before this commit: robot nanohand, 22 links, 21 joints
Links:
- added link index_fingertip
- added link middle_fingertip
- added link pinky_fingertip
- added link ring_fingertip
- added link thumb_fingertip
Joints:
- added joint index_fingertip_joint: type fixed, parent index_tip, child index_fingertip, origin xyz=-0.001 -0.002 -0.030 rpy=0 0 0
- added joint middle_fingertip_joint: type fixed, parent middle_tip, child middle_fingertip, origin xyz=0.000 -0.001 -0.031 rpy=0 0 0
- added joint pinky_fingertip_joint: type fixed, parent pinky_tip, child pinky_fingertip, origin xyz=0.002 -0.003 -0.027 rpy=0 0 0
- added joint ring_fingertip_joint: type fixed, parent ring_tip, child ring_fingertip, origin xyz=0.000 -0.007 -0.027 rpy=0 0 0
- added joint thumb_fingertip_joint: type fixed, parent thumb_tip, child thumb_fingertip, origin xyz=0.000 -0.023 -0.016 rpy=0 0 0
- joint pinky_wiggle: limit lower=-0.17 upper=0.26 effort=1.0 velocity=3.0 -> lower=-0.17 upper=0.17 effort=1.0 velocity=3.0
- joint ring_wiggle: limit lower=-0.2 upper=0.07 effort=1.0 velocity=3.0 -> lower=-0.2 upper=0.13 effort=1.0 velocity=3.0
